File: kicad/project/PWM_motor_speed_controller.kicad_pcb (KiCad board)
At the start: 2 copper layers, 100.5 x 80 mm, 19 parts, among them J1 Conn_01x02, M1 Motor_DC, Q1 Q_NMOS_GDS, SW1 SW_Push, SW2 SW_Push, SW3 SW_Push, SW4 SW_Push, U1 ATmega32A-P

Commit message: Update firmware, PCB, and documentation
Parts:
- added R6: 330, Resistor_THT:R_Axial_DIN0204_L3.6mm_D1.6mm_P7.62mm_Horizontal, F.Cu at (131.4, 132.7)
- added R7: 330, Resistor_THT:R_Axial_DIN0204_L3.6mm_D1.6mm_P7.62mm_Horizontal, F.Cu at (131.4, 139.1)
- added R8: 330, Resistor_THT:R_Axial_DIN0204_L3.6mm_D1.6mm_P7.62mm_Horizontal, F.Cu at (131.4, 146.1)
- added RV1: R_Potentiometer, Potentiometer_THT:Potentiometer_Bourns_3386P_Vertical, F.Cu at (120.0, 142.2)
- added U2: RC1602A-GHW-ESX, Display:RC1602A, F.Cu at (190.5, 111.1)
- added Y1: Crystal, Crystal:Crystal_HC49-U_Vertical, F.Cu at (99.7, 135.0)
- moved D4 35.2 mm to (194.3, 90.8)
- moved J1 29.1 mm to (179.7, 97.2)
- moved M1 21.8 mm to (200.7, 72.4)
Connections:
- U1 pad 22: unconnected-(U1-PC0-Pad22) -> Net-(U1-PC0)
- U1 pad 23: unconnected-(U1-PC1-Pad23) -> Net-(U1-PC1)
- U1 pad 24: unconnected-(U1-PC2-Pad24) -> Net-(U1-PC2)
- U1 pad 25: unconnected-(U1-PC3-Pad25) -> Net-(U1-PC3)
- U1 pad 26: unconnected-(U1-PC4-Pad26) -> Net-(U1-PC4)
- U1 pad 27: unconnected-(U1-PC5-Pad27) -> Net-(U1-PC5)
Routing:
- net GND: track 232.3 -> 378.2 mm, vias 0 -> 1
- net VCC: track 55.2 -> 165.3 mm
- net Net-(D4-K): track 74.9 -> 168.6 mm
- net Net-(U2-Vo): track 0.00 -> 85.3 mm
- net Net-(U1-PC5): track 0.00 -> 81.9 mm
- net Net-(U1-PC4): track 0.00 -> 80.0 mm
- net Net-(U1-PC3): track 0.00 -> 78.2 mm
- net Net-(U1-PC2): track 0.00 -> 76.4 mm
- net Net-(U2-A/VEE): track 0.00 -> 71.8 mm
- net Net-(U1-PC1): track 0.00 -> 64.4 mm
- net Net-(D4-A): track 30.7 -> 90.2 mm
- net Net-(U1-PC0): track 0.00 -> 58.7 mm
- net Net-(U1-PA1): track 59.4 -> 103.5 mm
- net Net-(U1-PA2): track 55.6 -> 94.3 mm
- net Net-(U1-PA0): track 51.7 -> 87.9 mm
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Other:
- board size 100.5 x 80 mm -> 171.7 x 110.9 mm
