File: kicad/project/PWM_motor_speed_controller.kicad_sch (KiCad schematic)
At the start: 20 parts, among them J1 Conn_01x02, M1 Motor_DC, Q1 Q_NMOS_GDS, SW1 SW_Push, SW2 SW_Push, SW3 SW_Push, SW4 SW_Push, U1 ATmega32A-P, Y1 Crystal

Commit message: Update firmware, PCB, and documentation
Parts:
- added R6, R7, R8: 330, Resistor_THT:R_Axial_DIN0204_L3.6mm_D1.6mm_P7.62mm_Horizontal, symbol Device:R
- added RV1: R_Potentiometer, Potentiometer_THT:Potentiometer_Bourns_3386P_Vertical, symbol Device:R_Potentiometer
- added U2: RC1602A-GHW-ESX, Display:RC1602A, symbol Display_Character:RC1602A-GHW-ESX
Connections:
- net GND: now also R6.1, R7.2, RV1.3, U2.1 (VSS), U2.16 (K), U2.5 (R/~{W})
- net VCC: now also R6.2, R8.1, RV1.1, U2.2 (VDD)
- net at U1.22 (PC0): now also U2.4 (RS)
- net at U1.23 (PC1): now also U2.6 (~{E})
- net at U1.24 (PC2): now also U2.11 (DB4)
- net at U1.25 (PC3): now also U2.12 (DB5)
- net at U1.26 (PC4): now also U2.13 (DB6)
- net at U1.27 (PC5): now also U2.14 (DB7)
- new net: R7.1, R8.2, U2.15 (A/VEE)
- new net: RV1.2, U2.3 (Vo)
